Commit message: Fix URDF viusal issues, remove redunant imu, and finalize robot hirarcy

File: install/amr_sqr_description/share/amr_sqr_description/description/camera.xacro (robot description, xacro)
@@ -1,7 +1,4 @@
 <?xml version="1.0"?>
 <robot xmlns:xacro="http://www.ros.org/wiki/xacro">
-    <material name="black">
-        <color rgba="0 0 0 1"/>
-    </material>
     <joint name="camera_joint" type="fixed">
         <parent link="base_link"/>
